File: teensy/mcu_to_tlc5947.kicad_pcb (KiCad board)
At the start: 2 copper layers, 152.4 x 76.2 mm, 14 parts, among them J1 conn_1x2, J2 conn_1x3, J3 conn_2x13_odd_even, J4 conn_2x3_odd_even, J5 conn_2x5_odd_even, J6 conn_2x5_odd_even, J7 conn_1x24, J8 conn_1x24, M1 VAL**, M2 VAL**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

Commit message: Fixed error with adafruit tlc5947 foot print.
Routing:
- net /PWM23: track 128.1 -> 163.4 mm
- net /PWM1: track 189.5 -> 158.1 mm
- net /PWM16: track 85.9 -> 113.8 mm
- net GND: track 253.3 -> 269.3 mm
- net /PWM19: track 141.5 -> 126.8 mm, vias 0 -> 1
- net /PWM10: track 96.0 -> 82.0 mm, vias 1 -> 2
- net /D0: track 44.4 -> 57.7 mm
- net /VIN: track 359.1 -> 371.8 mm
- net /PWM15: track 110.3 -> 97.8 mm, vias 0 -> 1
- net /PWM3: track 133.2 -> 122.4 mm
- net /PWM21: track 159.9 -> 149.3 mm
- net /PWM22: track 131.5 -> 121.6 mm
- net /PWM11: track 106.4 -> 97.9 mm
- net /PWM13: track 90.3 -> 98.4 mm, vias 0 -> 1
- net /PWM4: track 117.3 -> 110.6 mm
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Other:
- board text added: "Teensy-to-TLC5947 V0.2 Dickinson Lab 2018"
- board text removed: "Teensy-to-TLC5947 V0.1 Dickinson Lab 2018"
